File: KiCadTeensyFolkracePro.kicad_pcb (KiCad board)
At the start: 2 copper layers, 50.8 x 97.8 mm, 38 parts, among them P1 MOTOR, P2 STEERING, P3 START, U1 WS2812B, U10 GP2Y0E02B, U11 GP2Y0E02B, U12 GP2Y0E02B, U13 GP2Y0E02B, U2 Teensy31_32, U3 WS2812B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

Commit message: Arduino files
Parts:
- moved R1 109.4 mm to (104.1, 88.9), turned to 180 degrees
- moved R13 103.0 mm to (125.7, 138.4), turned to 90 degrees
- moved D1 101.0 mm to (109.2, 88.9)
- moved R14 101.0 mm to (123.2, 138.4), turned to 270 degrees
- moved R5 89.6 mm to (134.6, 111.1), turned to 180 degrees
- moved U4 88.8 mm to (115.6, 144.8), turned to 180 degrees
- moved R6 88.3 mm to (134.6, 113.7), turned to 180 degrees
- moved R16 87.3 mm to (130.8, 138.4), turned to 90 degrees
- moved R17 84.4 mm to (134.6, 130.2), turned to 180 degrees
- moved R3 82.7 mm to (127.0, 120.7)
- moved R8 81.1 mm to (134.6, 104.1), turned to 180 degrees
- moved R11 79.0 mm to (124.5, 94.6), turned to 270 degrees
- moved R19 78.8 mm to (134.6, 120.7), turned to 180 degrees
- moved R18 78.5 mm to (134.6, 133.3), turned to 180 degrees
- moved P1 74.0 mm to (106.0, 142.2), turned to 90 degrees
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Routing:
- net +3V3: track 0.00 -> 212.6 mm, vias 0 -> 10
- net GND: track 0.00 -> 166.1 mm, vias 0 -> 5
- net +5V: track 0.00 -> 101.8 mm, vias 0 -> 2
- net BT_TX: track 0.00 -> 63.4 mm
- net BT_RX: track 0.00 -> 62.9 mm, vias 0 -> 1
- net MOTOR: track 0.00 -> 41.9 mm
- net Net-(R16-Pad1): track 0.00 -> 35.8 mm, vias 0 -> 2
- net STEERING: track 0.00 -> 34.4 mm
- net Net-(R14-Pad1): track 0.00 -> 34.2 mm, vias 0 -> 2
- net Net-(R10-Pad1): track 0.00 -> 33.6 mm, vias 0 -> 2
- net Net-(R15-Pad1): track 0.00 -> 33.0 mm
- net Net-(R8-Pad1): track 0.00 -> 30.2 mm
- net Net-(R2-Pad1): track 0.00 -> 30.0 mm, vias 0 -> 2
- net Net-(R13-Pad1): track 0.00 -> 29.8 mm
- net STARTMODULE: track 0.00 -> 29.8 mm
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- added copper zone on F.Cu, net GND
Other:
- board size 50.8 x 97.8 mm -> 48.3 x 63.5 mm
- net class Power added: clearance 0.2, trace_width 0.3, via_dia 0.6, via_drill 0.4
- board text added: "Frode Lillerud 13.april 2016"
