File: KiCadTeensyFolkracePro.sch (KiCad schematic (older format))
At the start: 38 parts, among them P1 MOTOR, P2 STEERING, P3 START, U1 WS2812B, U10 GP2Y0E02B, U11 GP2Y0E02B, U12 GP2Y0E02B, U13 GP2Y0E02B, U2 Teensy31_32, U3 WS2812B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

Commit message: Changes
Parts:
- U1, U3: footprint (none) -> WS2812B:WS2812B
- U5: footprint (none) -> Housings_SSOP:TSSOP-24_4.4x7.8mm_Pitch0.65mm
Changed lines of the file:
@@
 F 0 "U5" H 6650 3900 60  0000 C CNN
 F 1 "TCA9548APWR" H 6650 2200 60  0000 C CNN
-F 2 "" H 6700 3450 60  0001 C CNN
+F 2 "Housings_SSOP:TSSOP-24_4.4x7.8mm_Pitch0.65mm" H 6700 3450 60  0001 C CNN
 F 3 "" H 6700 3450 60  0000 C CNN
 	1    6650 3300
@@
 F 0 "U3" H 3850 7000 60  0000 C CNN
 F 1 "WS2812B" H 3850 6400 60  0000 C CNN
-F 2 "" H 3800 6700 60  0001 C CNN
+F 2 "WS2812B:WS2812B" H 3800 6700 60  0001 C CNN
 F 3 "" H 3800 6700 60  0000 C CNN
 	1    3850 6700
@@
 F 0 "U1" H 2550 7000 60  0000 C CNN
 F 1 "WS2812B" H 2550 6400 60  0000 C CNN
-F 2 "" H 2500 6700 60  0001 C CNN
+F 2 "WS2812B:WS2812B" H 2500 6700 60  0001 C CNN
 F 3 "" H 2500 6700 60  0000 C CNN
 	1    2550 6700

Commit message: Schematic added
Parts:
- U10, U11, U12, U13, U6, U7, U8, U9: symbol GP2Y0E02B -> GP2Y0E02B-RESCUE-KiCadTeensyFolkracePro
Changed lines of the file:
@@
 EESchema Schematic File Version 2
+LIBS:KiCadTeensyFolkracePro-rescue
 LIBS:power
 LIBS:device
@@
 $EndComp
 $Comp
-L GP2Y0E02B U6
+L GP2Y0E02B-RESCUE-KiCadTeensyFolkracePro U6
 U 1 1 56F5200D
 P 10050 900
@@
 Connection ~ 8650 850
 $Comp
-L GP2Y0E02B U7
+L GP2Y0E02B-RESCUE-KiCadTeensyFolkracePro U7
 U 1 1 56F6346D
 P 10050 1600
@@
 Connection ~ 8650 1550
 $Comp
-L GP2Y0E02B U8
+L GP2Y0E02B-RESCUE-KiCadTeensyFolkracePro U8
 U 1 1 56F63959
 P 10050 2300
@@
 Connection ~ 8650 2250
 $Comp
-L GP2Y0E02B U9
+L GP2Y0E02B-RESCUE-KiCadTeensyFolkracePro U9
 U 1 1 56F63982
 P 10050 3000
@@
 Connection ~ 8650 2950
 $Comp
-L GP2Y0E02B U10
+L GP2Y0E02B-RESCUE-KiCadTeensyFolkracePro U10
 U 1 1 56F6459A
 P 10050 3700
@@
 Connection ~ 8650 3650
 $Comp
-L GP2Y0E02B U11
+L GP2Y0E02B-RESCUE-KiCadTeensyFolkracePro U11
 U 1 1 56F645C3
 P 10050 4400
@@
 Connection ~ 8650 4350
 $Comp
-L GP2Y0E02B U12
+L GP2Y0E02B-RESCUE-KiCadTeensyFolkracePro U12
 U 1 1 56F645EC
 P 10050 5100
@@
 Connection ~ 8650 5050
 $Comp
-L GP2Y0E02B U13
+L GP2Y0E02B-RESCUE-KiCadTeensyFolkracePro U13
 U 1 1 56F64615
 P 10050 5800
